File: hardware/kicad/PICkeeby.kicad_sch (KiCad schematic)
At the start: 35 parts, among them J1 PS/2 Connector, J2 PS/2 Connector, J3 MODE_SELECT, J4 Host Interface, J5 Conn_PIC_ICSP_ICD, J6 PS/2 Header, J7 PS/2 Header, U1 PIC16F18344-P, U2 74HCT574, U3 74HCT373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

Commit message: v2
Parts:
- removed D2: LED, LED_THT:LED_D3.0mm_FlatTop, symbol Device:LED
- removed R7: 470R, Resistor_THT:R_Axial_DIN0207_L6.3mm_D2.5mm_P10.16mm_Horizontal, symbol Device:R
- C1, C2, C3, C4, C5, C6, C7, C8: footprint Capacitor_THT:C_Disc_D6.0mm_W2.5mm_P5.00mm -> Capacitor_SMD:C_0805_2012Metric_Pad1.18x1.45mm_HandSolder
- R1, R10, R11, R2, R3, R4, R5, R6, R8, R9: footprint Resistor_THT:R_Axial_DIN0207_L6.3mm_D2.5mm_P10.16mm_Horizontal -> Resistor_SMD:R_0805_2012Metric_Pad1.20x1.40mm_HandSolder
- U2, U3: footprint Package_DIP:DIP-20_W7.62mm_Socket_LongPads -> Package_SO:SOIC-20W_7.5x12.8mm_P1.27mm
- renumbered D4 to D1, D5 to D2, D1 to D4
Connections:
- net VPP is gone; now on net A0: J5.1 (~{MCLR}/VPP), R1.2, U1.4 (RA3/~{MCLR}/VPP)
- net GND: no longer U4.8 (IN)
- net HDATA0: now also J4.9 (Pin_9); no longer J4.2 (Pin_2)
- net HDATA1: now also J4.8 (Pin_8); no longer J4.3 (Pin_3)
- net HDATA2: now also J4.7 (Pin_7); no longer J4.4 (Pin_4)
- net HDATA3: now also J4.6 (Pin_6); no longer J4.5 (Pin_5)
- net HDATA4: now also J4.5 (Pin_5); no longer J4.6 (Pin_6)
- net HDATA5: now also J4.4 (Pin_4), U4.21 (I/O); no longer J4.7 (Pin_7)
- net HDATA6: now also J4.3 (Pin_3); no longer J4.8 (Pin_8)
- net HDATA7: now also J4.2 (Pin_2); no longer J4.9 (Pin_9)
- net LED_RX: now also R8.2, U4.16 (I/O)
- net ~{AUX}: now also U4.8 (IN)
- net ~{RD_DATA}: now also U2.1 (OE)
Other:
- moved on the sheet: D4, R6

Commit message: v2
Parts:
- removed C2, C4, C6: 10nf, Capacitor_SMD:C_0805_2012Metric_Pad1.18x1.45mm_HandSolder, symbol Device:C
- removed C8: 10nF, Capacitor_SMD:C_0805_2012Metric_Pad1.18x1.45mm_HandSolder, symbol Device:C
- removed R1: 100K, Resistor_SMD:R_0805_2012Metric_Pad1.20x1.40mm_HandSolder, symbol Device:R
- added C5: 1µF, Capacitor_SMD:C_0805_2012Metric_Pad1.18x1.45mm_HandSolder, symbol Device:C
- added U5: 74AHCT1G14, Package_TO_SOT_SMD:SOT-23-5_HandSoldering, symbol 74xGxx:74AHCT1G14
- C1: value 100nF -> 1µF
- C2: renamed from C3; value 100nF -> 1µF
- C3: renamed from C5; value 100nF -> 1µF
- C4: renamed from C7; value 100nF -> 1µF
- R5: renamed from R9; value 470R -> 300Ω
- R6: renamed from R10; value 470R -> 300Ω
- R7: renamed from R8; value 470R -> 300Ω
- R8: renamed from R6; value 470R -> 300Ω
- U2: value 74HCT574 -> 74AHCT574
- U3: value 74HCT373 -> 74AHCT373
- renumbered R2 to R1, R3 to R2, R4 to R3, R5 to R4, R11 to R9
Connections:
- net +5V: now also J4.14 (Pin_14), R5.2, C5.1, U5.5 (VCC); no longer J4.1 (Pin_1)
- net A0: now also J4.9 (Pin_9); no longer J4.10 (Pin_10), J5.1 (~{MCLR}/VPP), U1.4 (RA3/~{MCLR}/VPP)
- net CLK_OUT: now also U4.9 (IN); no longer U4.1 (CLK/IN)
- net GND: now also C5.2, U5.3 (GND); no longer D1.1 (K), U4.9 (IN)
- net HDATA0: now also J4.8 (Pin_8), U3.3 (D0); no longer J4.9 (Pin_9), U3.2 (O0)
- net HDATA1: now also J4.7 (Pin_7), U3.4 (D1); no longer J4.8 (Pin_8), U3.5 (O1)
- net HDATA2: now also J4.6 (Pin_6), U3.7 (D2); no longer J4.7 (Pin_7), U3.6 (O2)
- net HDATA3: now also J4.5 (Pin_5), U3.8 (D3); no longer J4.6 (Pin_6), U3.9 (O3)
- net HDATA4: now also J4.4 (Pin_4), U3.13 (D4); no longer J4.5 (Pin_5), U3.12 (O4)
- net HDATA5: now also J4.3 (Pin_3), U3.14 (D5); no longer J4.4 (Pin_4), U3.15 (O5)
- net HDATA6: now also J4.2 (Pin_2), U3.17 (D6); no longer J4.3 (Pin_3), U3.16 (O6)
- net HDATA7: now also J4.1 (Pin_1), U3.18 (D7); no longer J4.2 (Pin_2), U3.19 (O7)
- net IDATA0: now also U3.2 (O0); no longer U3.3 (D0)
- net IDATA1: now also U3.5 (O1); no longer U3.4 (D1)
- net IDATA2: now also U3.6 (O2); no longer U3.7 (D2)
- net IDATA3: now also U3.9 (O3); no longer U3.8 (D3)
- net IDATA4: now also U3.12 (O4); no longer U3.13 (D4)
- net IDATA5: now also U3.15 (O5); no longer U3.14 (D5)
- net IDATA6: now also U3.16 (O6); no longer U3.17 (D6)
- net IDATA7: now also U3.19 (O7); no longer U3.18 (D7)
- net SIG1: now also J4.10 (Pin_10); no longer J4.11 (Pin_11)
- net SIG2: now also J4.11 (Pin_11), U5.2; no longer J4.13 (Pin_13)
- net ~{CS}: now also D1.1 (K)
- net ~{IRQ}: now also J4.13 (Pin_13); no longer J4.14 (Pin_14)
- net A0_REG: now reaches U4.14 (I/O)
- net A0_REG: now also U1.4 (RA3/~{MCLR}/VPP); no longer R5.2
- net LED_RX renamed IBF
- new net VPP: J5.1 (~{MCLR}/VPP)
- new net ~{SIG2}: U4.1 (CLK/IN), U5.4
Other:
- moved on the sheet: C1, C2, C3, C4, D1, R5

Commit message: GAL async reset for IBF clear, doc fixes, linting
- PLD: Add AR product term for async IBF/A0_REG clear (fixes Z80 deadlock)
- Firmware: Fix LATA init (OE_INB high at startup), simplify IBF clear
- Firmware: Move IDATA remap functions from pins.h to host.c
Connections:
- net A0: now also J4.10 (Pin_10); no longer J4.9 (Pin_9)
- net HDATA4: now also U3.18 (D7); no longer U3.13 (D4)
- net HDATA5: now also U3.17 (D6); no longer U3.14 (D5)
- net HDATA6: now also U3.14 (D5); no longer U3.17 (D6)
- net HDATA7: now also U3.13 (D4); no longer U3.18 (D7)
- net IDATA0: now also U1.5 (RC5); no longer U1.16 (RC0)
- net IDATA1: now also U1.16 (RC0); no longer U1.15 (RC1)
- net IDATA2: now also U1.6 (RC4); no longer U1.14 (RC2)
- net IDATA3: now also U1.15 (RC1); no longer U1.7 (RC3)
- net IDATA4: now also U1.7 (RC3), U3.19 (O7); no longer U1.6 (RC4), U3.12 (O4)
- net IDATA5: now also U1.14 (RC2), U3.16 (O6); no longer U1.5 (RC5), U3.15 (O5)
- net IDATA6: now also U3.15 (O5); no longer U3.16 (O6)
- net IDATA7: now also U3.12 (O4); no longer U3.19 (O7)
- net SIG1: now also J4.9 (Pin_9); no longer J4.10 (Pin_10)
